File: mcu_imu.kicad_sch (KiCad schematic)
At the start: 14 parts, among them IC5 ICM-20948, U3 STM32H745ZIT6, Y1 NX3215SA-32.768K-EXS00A-MU000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

Commit message: New structure for holding parts, symbols, and footprints
Parts:
- IC5: footprint ICM-20948:QFN40P300X300X105-25N-D -> CivicAlert:ICM-20948
- U3: footprint STM32H745ZIT6:LQFP-144 -> CivicAlert:STM32H745ZIT6
- Y1: footprint NX3215SA-32.768K:NX3215SA32768KEXS00AMU00003 -> CivicAlert:NX3215SA-32_768K-EXS00A-MU0000
Changed lines of the file:
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@@
 			)
 		)
-		(property "Footprint" "ICM-20948:QFN40P300X300X105-25N-D"
+		(property "Footprint" "CivicAlert:ICM-20948"
 			(at 15.57 172.72 0)
 			(effects
@@
 			)
 		)
-		(property "Footprint" "NX3215SA-32.768K:NX3215SA32768KEXS00AMU00003"
+		(property "Footprint" "CivicAlert:NX3215SA-32_768K-EXS00A-MU0000"
 			(at 82.88 69.85 0)
 			(effects
@@
 			)
 		)
-		(property "Footprint" "STM32H745ZIT6:LQFP-144"
+		(property "Footprint" "CivicAlert:STM32H745ZIT6"
 			(at 110.49 27.94 0)
 			(effects
