File: rpi.kicad_sch (KiCad schematic)
At the start: 4 parts, among them J4 10164227-1004A1RLF, J5 10164227-1004A1RLF

Commit message: New structure for holding parts, symbols, and footprints
Parts:
- J4, J5: footprint 10164227-1004A1RLF:AMPHENOL_10164227-1004A1RLF_NOPINS -> CivicAlert:10164227-1004A1RLF
- Module1: footprint RPI-CM5:Raspberry-Pi-5-Compute-Module -> CivicAlert:RPI-CM5IO
Changed lines of the file:
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@@
 			)
 		)
-		(property "Footprint" "RPI-CM5:Raspberry-Pi-5-Compute-Module"
+		(property "Footprint" "CivicAlert:RPI-CM5IO"
 			(at 196.85 119.38 0)
 			(effects
@@
 			)
 		)
-		(property "Footprint" "10164227-1004A1RLF:AMPHENOL_10164227-1004A1RLF_NOPINS"
+		(property "Footprint" "CivicAlert:10164227-1004A1RLF"
 			(at 29.21 92.71 0)
 			(effects
@@
 			)
 		)
-		(property "Footprint" "RPI-CM5:Raspberry-Pi-5-Compute-Module"
+		(property "Footprint" "CivicAlert:RPI-CM5IO"
 			(at 247.65 114.3 0)
 			(effects
@@
 			)
 		)
-		(property "Footprint" "10164227-1004A1RLF:AMPHENOL_10164227-1004A1RLF_NOPINS"
+		(property "Footprint" "CivicAlert:10164227-1004A1RLF"
 			(at 265.43 92.71 0)
 			(effects
