File: usb_debug.kicad_sch (KiCad schematic)
At the start: 32 parts, among them IC2 ESDALC6V1W5, IC3 ESDALC6V1W5, J7 USB4105-GF-A, Q3 BC847CE6327HTSA1, U3 STM32H745ZIT6, U8 TS3USB221RSER, Y2 ATX-H11-F-25.000MHz-F25-T

Commit message: New structure for holding parts, symbols, and footprints
Parts:
- B1: footprint 009159010061911:009159010061911 -> CivicAlert:009159010061911
- D1: footprint NSPM2051MUT5G:DIODFN160X100X55-2N -> CivicAlert:NSPM2051MUT5G
- IC2, IC3: footprint ESDALC6V1W5:SOT65P210X110-5N -> CivicAlert:ESDALC6V1W5
- Q3: footprint BC847CE6327HTSA1:PG-SOT23-3-1_INF -> CivicAlert:BC847CE6327HTSA1
- RESET1: footprint LS38G2F-T:SW-SMD_4P-L3.3-W3.1_LS38G2-T -> CivicAlert:LS38G2F-T
- U3: footprint STM32H745ZIT6:LQFP-144 -> CivicAlert:STM32H745ZIT6
- U8: footprint TS3USB221RSER:TS3USB221RSER -> CivicAlert:TS3USB221RSER
- USB1: footprint LTST-C193TBKT-5A:LED_LTST-C_LTO -> CivicAlert:LTST-C193TBKT-5A
- Y2: footprint ATX-H11-F-25.000MHZ-F25-T:ATXH11F25000MHzF25T -> CivicAlert:ATX-H11-F-25_000MHz-F25-T
Changed lines of the file:
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@@
 			)
 		)
-		(property "Footprint" "TS3USB221RSER:TS3USB221RSER"
+		(property "Footprint" "CivicAlert:TS3USB221RSER"
 			(at 187.96 147.32 0)
 			(effects
@@
 			)
 		)
-		(property "Footprint" "LS38G2F-T:SW-SMD_4P-L3.3-W3.1_LS38G2-T"
+		(property "Footprint" "CivicAlert:LS38G2F-T"
 			(at 154.94 63.5 0)
 			(effects
@@
 			)
 		)
-		(property "Footprint" "LTST-C193TBKT-5A:LED_LTST-C_LTO"
+		(property "Footprint" "CivicAlert:LTST-C193TBKT-5A"
 			(at 57.15 162.56 0)
 			(effects
@@
 			)
 		)
-		(property "Footprint" "009159010061911:009159010061911"
+		(property "Footprint" "CivicAlert:009159010061911"
 			(at 226.06 25.4 0)
 			(effects
@@
 			)
 		)
-		(property "Footprint" "STM32H745ZIT6:LQFP-144"
+		(property "Footprint" "CivicAlert:STM32H745ZIT6"
 			(at 45.72 35.56 0)
 			(effects
@@
 			)
 		)
-		(property "Footprint" "NSPM2051MUT5G:DIODFN160X100X55-2N"
+		(property "Footprint" "CivicAlert:NSPM2051MUT5G"
 			(at 137.16 73.66 0)
 			(effects
@@
 			)
 		)
-		(property "Footprint" "ESDALC6V1W5:SOT65P210X110-5N"
+		(property "Footprint" "CivicAlert:ESDALC6V1W5"
 			(at 203.2 150.8 0)
 			(effects
@@
 			)
 		)
-		(property "Footprint" "BC847CE6327HTSA1:PG-SOT23-3-1_INF"
+		(property "Footprint" "CivicAlert:BC847CE6327HTSA1"
 			(at 49.53 177.8 0)
 			(effects
@@
 			)
 		)
-		(property "Footprint" "ESDALC6V1W5:SOT65P210X110-5N"
+		(property "Footprint" "CivicAlert:ESDALC6V1W5"
 			(at 245.11 150.8 0)
 			(effects
@@
 			)
 		)
-		(property "Footprint" "ATX-H11-F-25.000MHZ-F25-T:ATXH11F25000MHzF25T"
+		(property "Footprint" "CivicAlert:ATX-H11-F-25_000MHz-F25-T"
 			(at 113.03 -33.96 0)
 			(effects
