File: hw.kicad_pcb (KiCad board)
At the start: 4 copper layers, 75 x 75 mm, 247 parts, among them IC1 MX25UM25645GXDI00-T, IC2 ESDALC6V1W5, IC3 ESDALC6V1W5, IC4 ICM-20948, J1 USB4105-GF-A, J2 78800-0001, Q1 SI1062X-T1-GE3, Q2 MMBT3904LT3G, Q3 MMBT3904LT3G, Q4 MMBT3904LT3G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

Commit message: Updates for Rev. C
Parts:
- removed C47, C48: 3.3p, Capacitor_SMD:C_0402_1005Metric
- removed C49: 10n, Capacitor_SMD:C_0402_1005Metric
- removed C50: 0.1u, Capacitor_SMD:C_0201_0603Metric
- removed FID1, FID2, FID3, FID4, FID5, FID6: Fiducial, Fiducial:Fiducial_1mm_Mask3mm
- removed Q2: MMBT3904LT3G, CivicAlert:MMBT3904LT3G
- removed R29: 300, Resistor_SMD:R_0402_1005Metric
- removed R30: 10k, Resistor_SMD:R_0402_1005Metric
- removed R31: 47k, Resistor_SMD:R_0402_1005Metric
- removed USB1: LTST-C190KGKT, CivicAlert:LTST-C190KGKT
- removed Y1: ABS07AIG-32.768KHZ-7-T, CivicAlert:ABS07AIG_32_768KHZ_7_T
- removed Y2: KC2016Z48.0000C15XXK, CivicAlert:KC2016Z48.0000C15XXK
- added F1: Fiducial, Fiducial:Fiducial_1mm_Mask3mm, F.Cu at (113.7, 62.7)
- added F2: Fiducial, Fiducial:Fiducial_1mm_Mask3mm, F.Cu at (185.1, 62.7)
- added F3: Fiducial, Fiducial:Fiducial_1mm_Mask3mm, F.Cu at (113.7, 134.1)
- added F4: Fiducial, Fiducial:Fiducial_1mm_Mask3mm, B.Cu at (113.7, 62.7)
- added F5: Fiducial, Fiducial:Fiducial_1mm_Mask3mm, B.Cu at (185.1, 62.7)
- added F6: Fiducial, Fiducial:Fiducial_1mm_Mask3mm, B.Cu at (113.7, 134.1)
- added H1: MountingHole, MountingHole:MountingHole_2.2mm_M2, F.Cu at (123.9, 65.8)
- added H2: MountingHole, MountingHole:MountingHole_2.2mm_M2, F.Cu at (115.1, 107.9)
- added H3: MountingHole, MountingHole:MountingHole_2.2mm_M2, F.Cu at (182.8, 103.8)
- added R63: 2.2k, Resistor_SMD:R_0402_1005Metric, B.Cu at (154.0, 88.5)
- added R64: 2.2k, Resistor_SMD:R_0402_1005Metric, F.Cu at (152.7, 86.7)
- C108, C109, C110, C111, CH1, CH2, CH3, CH4, R53, R54, R55, R56: moved to F.Cu
- CELL1, GPS1, PWR1, Q3, Q4, R10, R46, R47, R48, R50, R51, R52: moved to B.Cu
- J1: value USB4105-GF-A -> USB4730-GF-A_REVA; footprint Connector_USB:USB_C_Receptacle_GCT_USB4105-xx-A_16P_TopMnt_Horizontal -> CivicAlert:USB4730-GF-A
- R13: value 22 -> 10k; footprint Resistor_SMD:R_0201_0603Metric -> Resistor_SMD:R_0402_1005Metric
- R14: value 1k -> 10k; footprint Resistor_SMD:R_0201_0603Metric -> Resistor_SMD:R_0402_1005Metric
- R43, R44, R60, R61: value 10k -> 2.2k
- moved R50 6.29 mm to (179.2, 109.5)
- moved R46 5.98 mm to (179.2, 117.5)
- moved R14 5.76 mm to (164.0, 81.8), turned to -90 degrees
- moved R10 5.37 mm to (179.6, 101.0), turned to 0 degrees
- moved C110 4.92 mm to (114.5, 67.9), turned to -90 degrees
- moved PWR1 4.81 mm to (179.9, 99.8), turned to 180 degrees
- moved GPS1 4.80 mm to (180.0, 107.8), turned to 180 degrees
- moved C108 4.80 mm to (179.5, 66.9)
- moved R51 4.48 mm to (184.2, 111.6)
- moved CELL1 4.37 mm to (180.0, 115.8), turned to 180 degrees
- moved R47 4.04 mm to (184.2, 119.6)
- moved CR2 3.65 mm to (174.7, 131.8), turned to 0 degrees
- moved J1 2.10 mm to (149.4, 62.4)
- moved Q4 1.99 mm to (182.1, 109.6), turned to 180 degrees
- moved R52 1.99 mm to (182.1, 112.1), turned to 180 degrees
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Connections:
- R13 pad 1: Net-(Y2-OUTPUT) -> GND
- R14 pad 2: Net-(U6B-PH1-OSC_OUT) -> Net-(U6A-PC14-OSC32_IN)
- U12 pad 100: unconnected-(U12-VBCKP_GNSS-Pad100) -> GPS_VINT
- U6 pad B5: Net-(U6B-PH1-OSC_OUT) -> unconnected-(U6B-PH1-OSC_OUT-PadB5)
- U6 pad D1: Net-(U6A-PC15-OSC32_OUT) -> unconnected-(U6A-PC15-OSC32_OUT-PadD1)
- U6 pad D19: LED_MCU_STATUS -> unconnected-(U6A-PB6-PadD19)
- U6 pad W2: GND -> VCC_MCU_1V8
Routing:
- net GND: track 248.4 -> 204.0 mm, vias 592 -> 565
- net LED_MCU_STATUS: track 30.0 -> 0.00 mm
- net VCC_5V: track 234.6 -> 218.5 mm, vias 10 -> 14
- net LED_NETWORK: track 41.1 -> 50.1 mm, vias 0 -> 1
- net AI_BOOT_DEV: track 37.9 -> 31.9 mm, vias 6 -> 4
- net VCC_AI_ON: track 121.8 -> 116.2 mm
- net LED_GPS_STATUS: track 58.1 -> 62.1 mm, vias 2 -> 1
- net Net-(U6A-PC15-OSC32_OUT): track 3.44 -> 0.00 mm
- net Net-(Q2-Pad1): track 3.04 -> 0.00 mm
- net Net-(U6B-PH1-OSC_OUT): track 2.92 -> 0.00 mm, vias 2 -> 0
- net MIC_CLK1_2: track 94.7 -> 92.5 mm, vias 3 -> 4
- net Net-(U6A-PC14-OSC32_IN): track 3.45 -> 1.31 mm
- net VCC_MCU_1V8: track 323.6 -> 325.6 mm, vias 17 -> 19
- net GPS_VINT: track 42.4 -> 44.4 mm
- net Net-(Q2-Pad3): track 1.65 -> 0.00 mm
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Other:
- board text added: "Rev. C"
- board text removed: "Rev. B"
