File: ai_memory.kicad_sch (KiCad schematic)
At the start: 15 parts, among them IC1 MX25UM25645GXDI00-T, IC2 ESDALC6V1W5

Commit message: Finalize RevB
Parts:
- removed D1: B140Q-13-F, CivicAlert:B140Q-13-F, symbol B140Q-13-F:B140Q-13-F
- added BOOT1: PTS810, CivicAlert:PTS810, symbol PTS810:PTS810
- added CR6: BAT854W,115, CivicAlert:BAT854AW,115, symbol BAT854W,115:BAT854W_115
- added R62: 10k, Resistor_SMD:R_0402_1005Metric, symbol Device:R
- C51, C54, C55: MPN (none) -> GRM155R71C104KA88J
- C52, C53, C56: MPN (none) -> GRT155D70J475ME13D
Connections:
- net AI_BOOT_DEV: now also BOOT1.1, BOOT1.2, R62.2
- net AI_NRST: now also CR6.3
- net GND: now also R62.1
- net VCC_AI_IO: now also BOOT1.3, BOOT1.4
- net at IC1.A4 (RESET#), R15.1: now also CR6.1
Other:
- note added: "Boot Mode Switch"
- moved on the sheet: C51, C52, C53, C54, C55, C56, IC1, R15, R16, R17
