File: hw.kicad_sch (KiCad schematic)
At the start: 0 parts

Commit message: Update for RevB
Other:
- sheet MCU + IMU renamed IMU
- sheet USB + Debug renamed MCU Debug + USB
- removed sheet Raspberry Pi
- added sheet AI Clocks and GPIO (ai_gpio.kicad_sch)
- added sheet AI Memory + Debug (ai_memory.kicad_sch)
- added sheet AI System (ai_system.kicad_sch)
- added sheet MCU Clocks and GPIO (mcu_clocks_gpio.kicad_sch)
- added sheet MCU System (mcu_system.kicad_sch)
- added sheet SD Card (sd_card.kicad_sch)
- sheet IMU: file mcu_imu.kicad_sch -> imu.kicad_sch
- sheet MCU Debug + USB: file usb_debug.kicad_sch -> mcu_debug_usb.kicad_sch

Commit message: Updates for Rev. C
Other:
- added sheet Structural (structural.kicad_sch)
Changed lines of the file:
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@@
 	(title_block
 		(title "CivicAlert")
-		(date "2025-08-19")
-		(rev "B")
+		(date "2025-11-13")
+		(rev "C")
 		(company "Vanderbilt University")
 	)
@@
 	)
 	(sheet
-		(at 222.25 96.52)
+		(at 200.66 96.52)
 		(size 26.67 34.29)
 		(exclude_from_sim no)
@@
 		)
 		(property "Sheetname" "Audio"
-			(at 222.25 95.8084 0)
+			(at 200.66 95.8084 0)
 			(effects
 				(font
@@
 		)
 		(property "Sheetfile" "audio.kicad_sch"
-			(at 222.25 131.3946 0)
+			(at 200.66 131.3946 0)
 			(effects
 				(font
@@
 	)
 	(sheet
-		(at 135.89 96.52)
+		(at 114.3 96.52)
 		(size 26.67 34.29)
 		(exclude_from_sim no)
@@
 		)
 		(property "Sheetname" "IMU"
-			(at 135.89 95.8084 0)
+			(at 114.3 95.8084 0)
 			(effects
 				(font
@@
 		)
 		(property "Sheetfile" "imu.kicad_sch"
-			(at 135.89 131.3946 0)
+			(at 114.3 131.3946 0)
 			(effects
 				(font
@@
 				(path "/37690768-e2be-4a37-b8f7-45d5da107609"
 					(page "10")
+				)
+			)
+		)
+	)
+	(sheet
+		(at 243.84 96.52)
+		(size 26.67 34.29)
+		(exclude_from_sim no)
+		(in_bom yes)
+		(on_board yes)
+		(dnp no)
+		(fields_autoplaced yes)
+		(stroke
+			(width 0.1524)
+			(type solid)
+		)
+		(fill
+			(color 0 0 0 0.0000)
+		)
+		(property "Sheetname" "Structural"
+			(at 243.84 95.8084 0)
+			(effects
+				(font
+					(size 1.27 1.27)
+				)
+				(justify left bottom)
+			)
+		)
+		(property "Sheetfile" "structural.kicad_sch"
+			(at 243.84 131.3946 0)
+			(effects
+				(font
+					(size 1.27 1.27)
+				)
+				(justify left top)
+			)
+		)
+		(instances
+			(project "hw"
+				(path "/37690768-e2be-4a37-b8f7-45d5da107609"
+					(page "13")
 				)
 			)
@@
 	)
 	(sheet
-		(at 179.07 96.52)
+		(at 157.48 96.52)
 		(size 26.67 34.29)
 		(exclude_from_sim no)
@@
 		)
 		(property "Sheetname" "GPS + Cellular"
-			(at 179.07 95.8084 0)
+			(at 157.48 95.8084 0)
 			(effects
 				(font
@@
 		)
 		(property "Sheetfile" "gps_cellular.kicad_sch"
-			(at 179.07 131.3946 0)
+			(at 157.48 131.3946 0)
 			(effects
 				(font
@@
 	)
 	(sheet
-		(at 49.53 96.52)
+		(at 27.94 96.52)
 		(size 26.67 34.29)
 		(exclude_from_sim no)
@@
 		)
 		(property "Sheetname" "MCU Clocks and GPIO"
-			(at 49.53 95.8084 0)
+			(at 27.94 95.8084 0)
 			(effects
 				(font
@@
 		)
 		(property "Sheetfile" "mcu_clocks_gpio.kicad_sch"
-			(at 49.53 131.3946 0)
+			(at 27.94 131.3946 0)
 			(effects
 				(font
@@
 	)
 	(sheet
-		(at 93.98 96.52)
+		(at 72.39 96.52)
 		(size 26.67 34.29)
 		(exclude_from_sim no)
@@
 		)
 		(property "Sheetname" "MCU Debug + USB"
-			(at 93.98 95.8084 0)
+			(at 72.39 95.8084 0)
 			(effects
 				(font
@@
 		)
 		(property "Sheetfile" "mcu_debug_usb.kicad_sch"
-			(at 93.98 131.3946 0)
-			(effects
-				(font
+			(at 72.39 131.3946 0)
+			(effects
+				(font
