File: imu.kicad_sch (KiCad schematic)
At the start: 7 parts, among them IC4 ICM-20948

Commit message: Finalize RevB
Parts:
- C89, C90, C91: MPN (none) -> GRM155R71C104KA88J
Connections:
- net VCC_MCU renamed VCC_MCU_1V8

Commit message: Updates for Rev. C
Parts:
- R43, R44: value 10k -> 2.2k
Changed lines of the file:
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@@
 	(title_block
 		(title "CivicAlert")
-		(date "2025-08-19")
-		(rev "B")
+		(date "2025-11-13")
+		(rev "C")
 		(company "Vanderbilt University")
 	)
@@
 			)
 		)
-		(property "Value" "10k"
+		(property "Value" "2.2k"
 			(at 196.85 87.6299 0)
 			(effects
@@
 			)
 		)
-		(property "Value" "10k"
+		(property "Value" "2.2k"
 			(at 177.8 87.6299 0)
 			(effects
