File: mcu_clocks_gpio.kicad_sch (KiCad schematic)
At the start: 15 parts, among them U11 STM32H745ZIT6, Y3 ATX-H11-F-25.000MHz-F25-T, Y4 ABS07AIG-32.768KHZ-7-T

Commit message: Finalize RevB
Parts:
- C82: MPN (none) -> GCM155R71H103KA55D
- C83, C85: MPN (none) -> GRM155R71C104KA88J
- C84, C86: MPN (none) -> GRT1555C1H3R3CA02J
- U11: MPN (none) -> STM32H745ZIT6
- Y4: MPN (none) -> ABS07AIG-32.768KHZ-7-T; Manufacturer (none) -> Abracon
Connections:
- net VCC_MCU: no longer C82.1, C83.1, Y3.1 (~{INH}), Y3.4 (VDD)
- new net VCC_MCU_1V8: C82.1, C83.1, Y3.1 (~{INH}), Y3.4 (VDD)

Commit message: Updates for Rev. C
Changed lines of the file:
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@@
 	(title_block
 		(title "CivicAlert")
-		(date "2025-08-19")
-		(rev "B")
+		(date "2025-11-13")
+		(rev "C")
 		(company "Vanderbilt University")
 	)
@@
 		(dnp no)
 		(property "Reference" "R32"
-			(at 226.06 71.12 90)
+			(at 226.06 75.946 90)
 			(effects
 				(font
@@
 		)
 		(property "Value" "22"
-			(at 226.06 68.58 90)
-			(effects
-				(font
+			(at 226.06 71.628 90)
+			(effects
+				(font
