File: mcu_system.kicad_sch (KiCad schematic)
At the start: 28 parts, among them Q2 MMBT3904LT3G, U11 STM32H745ZIT6

Commit message: Finalize RevB
Parts:
- C62, C76, C79: MPN (none) -> GRT155D70J475ME13D
- C63, C64, C65, C66, C67, C68, C69, C70, C71, C72, C73, C74, C75, C77: MPN (none) -> GRM155R71C104KA88J
- C78, C80, C81: MPN (none) -> GRT155C71A225KE13D
- FL1: MPN (none) -> FCM1608KF-601T03
- Q2: MPN (none) -> BC847CE6327HTSA1
- U11: MPN (none) -> STM32H745ZIT6
- USB1: MPN (none) -> LTST-C190KGKT
Connections:
- net VCC_3V3: no longer names the net of C78.1, U11.91 (VDD33USB)

Commit message: Updates for Rev. C
Parts:
- removed Q2: MMBT3904LT3G, CivicAlert:MMBT3904LT3G, symbol MMBT3904LT3G:BC847CE6327HTSA1
- removed R29: 300, Resistor_SMD:R_0402_1005Metric, symbol Device:R
- removed R30: 10k, Resistor_SMD:R_0402_1005Metric, symbol Device:R
- removed R31: 47k, Resistor_SMD:R_0402_1005Metric, symbol Device:R
- removed USB1: LTST-C190KGKT, CivicAlert:LTST-C190KGKT, symbol LTST-C190KGKT:LTST-C190KGKT
Other:
- note removed: "MCU Status LED"
- moved on the sheet: C62, C63, C64, C65, C66, C67, C68, C69, C70, C71, C72, C73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
