File: ai_gpio.kicad_sch (KiCad schematic)
At the start: 10 parts, among them U6 STM32N647L0H3Q, Y1 ABS07AIG-32.768KHZ-7-T, Y2 KC2016Z48.0000C15XXK

Commit message: Finalize RevB
Parts:
- C47, C48: MPN (none) -> GRT1555C1H3R3CA02J
- C49: MPN (none) -> GCM155R71H103KA55D
- C50: MPN (none) -> GRM033Z71C104KE14D
- U6: MPN (none) -> STM32N647L0H3Q; Manufacturer (none) -> STMicroelectronics
- Y1: MPN (none) -> ABS07AIG-32.768KHZ-7-T; Manufacturer (none) -> Abracon
- Y2: MANUFACTURER Kyocera -> (none); MAXIMUM_PACKAGE_HEIGHT 0.80mm -> (none); MPN (none) -> KC2016Z48.0000C15XXK; Manufacturer (none) -> Kyocera; PARTREV August 2021 -> (none); SNAPEDA_PN KC2016Z2.04800C1KX00 -> (none); STANDARD Manufacturer Recommendations -> (none)

Commit message: Updates for Rev. C
Parts:
- removed C47, C48: 3.3p, Capacitor_SMD:C_0402_1005Metric, symbol Device:C
- removed C49: 10n, Capacitor_SMD:C_0402_1005Metric, symbol Device:C
- removed C50: 0.1u, Capacitor_SMD:C_0201_0603Metric, symbol Device:C
- removed Y1: ABS07AIG-32.768KHZ-7-T, CivicAlert:ABS07AIG_32_768KHZ_7_T, symbol ABS07AIG-32.768KHZ-7-T:ABS07AIG-32.768KHZ-7-T
- removed Y2: KC2016Z48.0000C15XXK, CivicAlert:KC2016Z48.0000C15XXK, symbol KC2016Z48.0000C15XXK:KC2016Z48.0000C15XXK
- added R63, R64: 2.2k, Resistor_SMD:R_0402_1005Metric, symbol Device:R
- R13: value 22 -> 10k; footprint Resistor_SMD:R_0201_0603Metric -> Resistor_SMD:R_0402_1005Metric
- R14: value 1k -> 10k; footprint Resistor_SMD:R_0201_0603Metric -> Resistor_SMD:R_0402_1005Metric
Connections:
- net AI_DATA_OUT_SCL: now also R64.1
- net AI_DATA_OUT_SDA: now also R63.1
- net GND: now also R13.1
- net at U6.E1 (PC14-OSC32_IN): now also R14.2
- net at U6.B5 (PH1-OSC_OUT): no longer R14.2
- net LED_MCU_STATUS: no longer names the net of U6.D19 (PB6)
- new net VCC_MCU_1V8: R63.2, R64.2
- no-connect marks 86 -> 89
Other:
- moved on the sheet: R12, R13, R14, U6A, U6B

Commit message: Update RevC design
Connections:
- net AI_OVERDRIVE: no longer names the net of U6.V1 (PF13)
- no-connect marks 89 -> 90
Changed lines of the file:
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@@
+	)
+	(no_connect
+		(at 181.61 118.11)
 	)
 	(no_connect
@@
 		(pts
 			(xy 40.64 72.39) (xy 40.64 73.66)
-		)
-		(stroke
-			(width 0)
-			(type default)
-		)
-	)
-	(wire
-		(pts
-			(xy 179.07 118.11) (xy 181.61 118.11)
 		)
 		(stroke
@@
 			(effects
 				(font
-					(size 1.27 1.27)
-				)
-				(justify right)
-				(hide yes)
-			)
-		)
-	)
-	(global_label "AI_OVERDRIVE"
-		(shape output)
-		(at 179.07 118.11 180)
-		(fields_autoplaced yes)
-		(effects
-			(font
-				(size 1.27 1.27)
-			)
-			(justify right)
-		)
-		(property "Intersheetrefs" "${INTERSHEET_REFS}"
-			(at 163.2033 118.11 0)
-			(effects
-				(font
