File: mcu_debug_usb.kicad_sch (KiCad schematic)
At the start: 9 parts, among them IC3 ESDALC6V1W5, J1 USB4105-GF-A

Commit message: Finalize RevB
Parts:
- C87, C88: MPN (none) -> GRM155R71C104KA88J
Connections:
- net VCC_MCU renamed VCC_MCU_1V8
Other:
- moved on the sheet: B2, IC3, R39, R40

Commit message: Updates for Rev. C
Parts:
- removed J1: USB4105-GF-A, Connector_USB:USB_C_Receptacle_GCT_USB4105-xx-A_16P_TopMnt_Horizontal, symbol Connector:USB_C_Receptacle_USB2.0_16P
- added J1: USB4730-GF-A_REVA, CivicAlert:USB4730-GF-A, symbol USB4730-GF-A:USB4730-GF-A_REVA
Connections:
- net GND: now also J1.A1/B12 (GND_A), J1.B1/A12 (GND_B), J1.SH1 (SHELL_GND), J1.SH2 (SHELL_GND), J1.SH3 (SHELL_GND), J1.SH4 (SHELL_GND)
- net USB_D+: now also J1.A6 (DP1), J1.B6 (DP2)
- net USB_D-: now also J1.A7 (DN1), J1.B7 (DN2)
- net VCC_5V: now also J1.A4/B9 (VBUS_A), J1.B4/A9 (VBUS_B)
- net at R42.2: now also J1.B5 (CC2)
- net at R41.2: now also J1.A5 (CC1)
Other:
- moved on the sheet: C87, C88, R41, R42

Commit message: Update RevC design
Parts:
- removed J1: USB4730-GF-A_REVA, CivicAlert:USB4730-GF-A, symbol USB4730-GF-A:USB4730-GF-A_REVA
- added J1: USB4730-GF-A, CivicAlert:USB4730-GF-A, symbol USB4730-GF-A:USB4730-GF-A
Connections:
- net GND: now also J1.A1/B12 (GND_A), J1.B1/A12 (GND_B), J1.SH1 (SHELL_GND), J1.SH2 (SHELL_GND), J1.SH3 (SHELL_GND), J1.SH4 (SHELL_GND)
- net USB_D+: now also J1.A6 (DP1), J1.B6 (DP2)
- net USB_D-: now also J1.A7 (DN1), J1.B7 (DN2)
- net VCC_5V: now also J1.A4/B9 (VBUS_A), J1.B4/A9 (VBUS_B)
- net at R42.2: now also J1.B5 (CC2)
- net at R41.2: now also J1.A5 (CC1)
Changed lines of the file:
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@@
-	)
-	(symbol
-		(lib_id "USB4730-GF-A:USB4730-GF-A_REVA")
-		(at 140.97 125.73 0)
-		(unit 1)
-		(exclude_from_sim no)
-		(in_bom yes)
-		(on_board yes)
-		(dnp no)
-		(fields_autoplaced yes)
-		(property "Reference" "J1"
-			(at 140.97 107.95 0)
-			(effects
-				(font
-					(size 1.27 1.27)
-				)
-			)
-		)
-		(property "Value" "USB4730-GF-A_REVA"
-			(at 140.97 110.49 0)
-			(effects
-				(font
-					(size 1.27 1.27)
-				)
-			)
-		)
-		(property "Footprint" "CivicAlert:USB4730-GF-A"
-			(at 140.97 125.73 0)
-			(effects
-				(font
-					(size 1.27 1.27)
-				)
-				(justify bottom)
-				(hide yes)
-			)
-		)
-		(property "Datasheet" ""
-			(at 140.97 125.73 0)
-			(effects
-				(font
-					(size 1.27 1.27)
-				)
-				(hide yes)
-			)
-		)
-		(property "Description" ""
-			(at 140.97 125.73 0)
-			(effects
-				(font
-					(size 1.27 1.27)
-				)
-				(hide yes)
-			)
-		)
-		(property "MF" "Global Connector Technology"
-			(at 140.97 125.73 0)
-			(effects
-				(font
-					(size 1.27 1.27)
-				)
-				(justify bottom)
-				(hide yes)
-			)
-		)
-		(property "MAXIMUM_PACKAGE_HEIGHT" "4.66mm"
-			(at 140.97 125.73 0)
-			(effects
-				(font
-					(size 1.27 1.27)
-				)
-				(justify bottom)
-				(hide yes)
-			)
-		)
-		(property "Package" "None"
-			(at 140.97 125.73 0)
-			(effects
-				(font
-					(size 1.27 1.27)
-				)
-				(justify bottom)
-				(hide yes)
-			)
-		)
-		(property "Price" "None"
-			(at 140.97 125.73 0)
-			(effects
-				(font
-					(size 1.27 1.27)
-				)
-				(justify bottom)
-				(hide yes)
-			)
-		)
-		(property "Check_prices" "https://www.snapeda.com/parts/USB4730-GF-A/Global+Connector+Technology/view-part/?ref=eda"
-			(at 140.97 125.73 0)
-			(effects
-				(font
-					(size 1.27 1.27)
-				)
-				(justify bottom)
-				(hide yes)
-			)
-		)
-		(property "STANDARD" "Manufacturer Recommendations"
-			(at 140.97 125.73 0)
-			(effects
-				(font
-					(size 1.27 1.27)
-				)
-				(justify bottom)
-				(hide yes)
-			)
-		)
-		(property "PARTREV" "A"
-			(at 140.97 125.73 0)
-			(effects
-				(font
-					(size 1.27 1.27)
-				)
-				(justify bottom)
-				(hide yes)
-			)
-		)
-		(property "SnapEDA_Link" "https://www.snapeda.com/parts/USB4730-GF-A/Global+Connector+Technology/view-part/?ref=snap"
-			(at 140.97 125.73 0)
-			(effects
-				(font
-					(size 1.27 1.27)
-				)
-				(justify bottom)
-				(hide yes)
-			)
-		)
-		(property "MP" "USB4730-GF-A"
-			(at 140.97 125.73 0)
-			(effects
-				(font
-					(size 1.27 1.27)
-				)
-				(justify bottom)
-				(hide yes)
-			)
-		)
-		(property "Description_1" "USB-C (USB TYPE-C) USB 2.0 Receptacle Connector 24 (16+8 Dummy) Position Surface Mount, Right Angle; Through Hole"
-			(at 140.97 125.73 0)
-			(effects
-				(font
-					(size 1.27 1.27)
-				)
-				(justify bottom)
-				(hide yes)
-			)
-		)
-		(property "MANUFACTURER" "Global Connector Technology"
-			(at 140.97 125.73 0)
-			(effects
-				(font
-					(size 1.27 1.27)
-				)
-				(justify bottom)
-				(hide yes)
-			)
-		)
-		(property "Availability" "In Stock"
-			(at 140.97 125.73 0)
-			(effects
-				(font
-					(size 1.27 1.27)
-				)
-				(justify bottom)
-				(hide yes)
-			)
-		)
-		(property "SNAPEDA_PN" "USB4730-GF-A"
-			(at 140.97 125.73 0)
-			(effects
-				(font
-					(size 1.27 1.27)
-				)
-				(justify bottom)
-				(hide yes)
-			)
-		)
-		(pin "A8"
-		)
-		(pin "A1/B12"
-		)
-		(pin "A7"
-		)
-		(pin "A6"
-		)
-		(pin "SH2"
-		)
-		(pin "A5"
-		)
-		(pin "B7"
-		)
-		(pin "SH3"
-		)
-		(pin "B5"
-		)
-		(pin "B6"
-		)
-		(pin "SH1"
-		)
-		(pin "A4/B9"
-		)
-		(pin "SH4"
-		)
-		(pin "B4/A9"
-		)
-		(pin "B8"
-		)
-		(pin "B1/A12"
-		)
-		(instances
-			(project ""
-				(path "/37690768-e2be-4a37-b8f7-45d5da107609/f1627d13-9b14-4928-99f6-c027237993a1"
-					(reference "J1")
-					(unit 1)
-				)
-			)
-		)
 	)
 	(symbol
@@
 					(unit 1)
 				)
+			)
+		)
+	)
+	(symbol
+		(lib_id "USB4730-GF-A:USB4730-GF-A")
+		(at 140.97 125.73 0)
+		(unit 1)
+		(exclude_from_sim no)
+		(in_bom yes)
+		(on_board yes)
+		(dnp no)
+		(fields_autoplaced yes)
+		(property "Reference" "J1"
+			(at 140.97 107.95 0)
+			(effects
+				(font
+					(size 1.27 1.27)
+				)
+			)
+		)
+		(property "Value" "USB4730-GF-A"
+			(at 140.97 110.49 0)
+			(effects
+				(font
+					(size 1.27 1.27)
+				)
+			)
+		)
+		(property "Footprint" "CivicAlert:USB4730-GF-A"
+			(at 140.97 125.73 0)
+			(effects
+				(font
+					(size 1.27 1.27)
+				)
+				(justify bottom)
+				(hide yes)
+			)
+		)
+		(property "Datasheet" ""
+			(at 140.97 125.73 0)
+			(effects
+				(font
+					(size 1.27 1.27)
+				)
+				(hide yes)
+			)
+		)
+		(property "Description" "USB4730-GF-A"
+			(at 140.97 125.73 0)
+			(effects
+				(font
+					(size 1.27 1.27)
+				)
+				(hide yes)
+			)
+		)
+		(property "Manufacturer" "Global Connector Technology"
+			(at 140.97 125.73 0)
+			(effects
+				(font
+					(size 1.27 1.27)
+				)
+				(justify bottom)
+				(hide yes)
+			)
+		)
+		(pin "B4/A9"
+		)
+		(pin "A4/B9"
+		)
+		(pin "B6"
+		)
+		(pin "B5"
+		)
+		(pin "B1/A12"
+		)
+		(pin "B7"
+		)
+		(pin "B8"
+		)
+		(pin "A1/B12"
+		)
+		(pin "A8"
+		)
+		(pin "A7"
+		)
+		(pin "A6"
+		)
+		(pin "A5"
+		)
+		(pin "SH4"
+		)
+		(pin "SH3"
+		)
+		(pin "SH2"
+		)
+		(pin "SH1"
+		)
+		(instances
+			(project ""
+				(path "/37690768-e2be-4a37-b8f7-45d5da107609/f1627d13-9b14-4928-99f6-c027237993a1"
+					(reference "J1")
+					(unit 1)
+				)
