File: structural.kicad_sch (KiCad schematic)
At the start: 9 parts

Commit message: Update RevC design
Parts:
- H1, H2, H3: footprint MountingHole:MountingHole_2.2mm_M2 -> CivicAlert:MountingHole_2.4mm_M2
Changed lines of the file:
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@@
 			)
 		)
-		(property "Footprint" "MountingHole:MountingHole_2.2mm_M2"
+		(property "Footprint" "CivicAlert:MountingHole_2.4mm_M2"
 			(at 166.37 111.76 0)
 			(effects
@@
 			)
 		)
-		(property "Footprint" "MountingHole:MountingHole_2.2mm_M2"
+		(property "Footprint" "CivicAlert:MountingHole_2.4mm_M2"
 			(at 214.63 111.76 0)
 			(effects
@@
 			)
 		)
-		(property "Footprint" "MountingHole:MountingHole_2.2mm_M2"
+		(property "Footprint" "CivicAlert:MountingHole_2.4mm_M2"
 			(at 190.5 111.76 0)
 			(effects
